File: Schematics/CAN-Interface-Board.kicad_pcb (KiCad board)
At the start: 4 copper layers, 50 x 100 mm, 70 parts, among them CN1 Limit Switch Connector 1, CN2 Limit Switch Connector 2, J1 Microsemi_FlashPro-JTAG-10, J2 USB_C_Receptacle, J3 Micro_SD_Card, J4 Screw_Terminal_01x02, J5 Screw_Terminal_01x02, J6 Conn_01x05_Pin, U1 SN65HVD230, U2 LDL1117-3.3, U3 STM32F405RGT6, U5 LSM6DS3TR-C, U7 Bosch BMP388, Y1 8mhz

Commit message: V2, need to add flash mem, and encoder
Parts:
- added C26: 100nf, Capacitor_SMD:C_0805_2012Metric_Pad1.18x1.45mm_HandSolder, F.Cu at (97.2, 73.6)
- added J7: Conn_01x04_Pin, Connector_JST:JST_PH_B4B-PH-K_1x04_P2.00mm_Vertical, F.Cu at (134.5, 117.0)
- added R17: 10k, Resistor_SMD:R_0805_2012Metric_Pad1.20x1.40mm_HandSolder, F.Cu at (92.4, 67.0)
- added R18: 10k, Resistor_SMD:R_0805_2012Metric_Pad1.20x1.40mm_HandSolder, F.Cu at (92.4, 69.9)
- added R31: 10k, Resistor_SMD:R_0805_2012Metric_Pad1.20x1.40mm_HandSolder, F.Cu at (92.4, 72.9)
- added U8: W25Q128JVP, Package_SON:WSON-8-1EP_6x5mm_P1.27mm_EP3.4x4.3mm, F.Cu at (99.0, 68.8)
- moved G*** 6.35 mm to (137.5, 107.5)
Connections:
- C1 pad 1: /USB5V -> GND
- C1 pad 2: GND -> /USB5V
- J2 pad S1: unconnected-(J2-SHIELD-PadS1)_3 -> (no net)
- J3 pad 3: /FlashSD/SDMISO -> /FlashSD/SDMOSI
- J3 pad 7: /FlashSD/SDMOSI -> /FlashSD/SDMISO
- U3 pad 37: /MCU/CurrentCheck -> /MCU/Encoder-B
- U3 pad 38: unconnected-(U3-PC7-Pad38) -> /MCU/Encoder-A
Routing:
- net /FlashSD/SDMISO: track 39.0 -> 41.8 mm
- net /USB5V: track 64.3 -> 66.5 mm, vias 0 -> 1
- net GND: track 120.8 -> 118.5 mm, vias 55 -> 54
- net /FlashSD/SDMOSI: track 39.0 -> 37.4 mm

Commit message: need to finish st link and flash mem layout
Parts:
- moved C26 46.1 mm to (126.5, 38.0), turned to 180 degrees
- moved U8 35.2 mm to (125.0, 45.0)
- moved C22 11.5 mm to (121.0, 27.5)
- moved J7 6.32 mm to (140.5, 119.0), turned to 180 degrees
- moved J1 2.18 mm to (129.0, 32.4), turned to -90 degrees
Connections:
- U3 pad 33: /CAN Transciever/CAN_TX_2 -> /CAN Transciever/CAN_RX_2
- U3 pad 34: /CAN Transciever/CAN_RX_2 -> /CAN Transciever/CAN_TX_2
Routing:
- net /MCU/Encoder-A: track 0.00 -> 52.8 mm, vias 0 -> 1
- net /MCU/Encoder-B: track 0.00 -> 48.7 mm, vias 0 -> 1
- net /MCU/NRST: track 59.4 -> 41.3 mm
- net /MCU/SWCLK: track 60.8 -> 43.4 mm
- net /MCU/SWDIO: track 56.9 -> 44.4 mm
- net /CAN Transciever/CAN_TX_2: track 37.0 -> 41.4 mm
- net +3.3V: track 83.9 -> 79.6 mm, vias 23 -> 22
- net GND: track 118.5 -> 117.4 mm, vias 54 -> 53
- net /CAN Transciever/CAN_RX_2: track 34.0 -> 34.6 mm
