File: Schematics/CAN-Interface-Board.kicad_pcb (KiCad board)
At the start: 4 copper layers, 50 x 100 mm, 76 parts, among them CN1 Limit Switch Connector 1, CN2 Limit Switch Connector 2, J1 Microsemi_FlashPro-JTAG-10, J2 USB_C_Receptacle, J3 Micro_SD_Card, J4 Screw_Terminal_01x02, J5 Screw_Terminal_01x02, J6 Conn_01x05_Pin, J7 Conn_01x04_Pin, U1 SN65HVD230, U2 LDL1117-3.3, U3 STM32F405RGT6, U5 LSM6DS3TR-C, U7 Bosch BMP388, U8 W25Q128JVP, Y1 8mhz

Commit message: pcb pending review and order
Parts:
- removed J3: Micro_SD_Card, Connector_Card:microSD_HC_Molex_47219-2001
- removed R8: 33r, Resistor_SMD:R_0805_2012Metric_Pad1.20x1.40mm_HandSolder
- removed R9: 10k, Resistor_SMD:R_0805_2012Metric_Pad1.20x1.40mm_HandSolder
- added J8: Micro_SD_Card, Connector_Card:microSD_HC_Molex_47219-2001, F.Cu at (117.8, 72.5)
- added R15: 10k, Resistor_SMD:R_0805_2012Metric_Pad1.20x1.40mm_HandSolder, F.Cu at (124.2, 62.4)
- J1: value Microsemi_FlashPro-JTAG-10 -> Conn_ARM_JTAG_SWD_10
- moved C26 48.5 mm to (129.0, 36.9), turned to 90 degrees
- moved R18 48.1 mm to (131.0, 41.2), turned to 90 degrees
- moved R31 45.6 mm to (121.3, 37.6), turned to -90 degrees
- moved U8 38.4 mm to (126.4, 41.9)
- moved R17 37.6 mm to (120.9, 42.4), turned to 180 degrees
- moved C22 3.12 mm to (127.9, 32.8), turned to -90 degrees
- moved J7 3.05 mm to (137.4, 117.8)
- moved G*** 2.51 mm to (140.0, 107.7)
- moved C5 2.49 mm to (131.3, 94.7)
- moved U2 2.15 mm to (128.6, 99.5)
- moved G*** 2.10 mm to (138.2, 90.9)
- moved J1 1.31 mm to (125.6, 32.0), turned to -90 degrees
- moved C1 0.40 mm to (126.9, 80.5), turned to -90 degrees
Connections:
- J1 pad 1: /MCU/SWCLK -> +3.3V
- J1 pad 10: GND -> /MCU/NRST
- J1 pad 2: GND -> /MCU/SWDIO
- J1 pad 3: unconnected-(J1-TDO-Pad3) -> GND
- J1 pad 4: unconnected-(J1-PGM/NC-Pad4) -> /MCU/SWCLK
- J1 pad 5: /MCU/SWDIO -> GND
- J1 pad 6: +3.3V -> /MCU/SWO
- J1 pad 8: /MCU/NRST -> unconnected-(J1-NC/TDI-Pad8)
- J1 pad 9: unconnected-(J1-TDI-Pad9) -> GND
- U2 pad 1: Net-(D1-K) -> GND
- U2 pad 2: GND -> +3.3V
- U2 pad 3: +3.3V -> Net-(D1-K)
- U3 pad 10: /FlashSD/SDMISO -> /FlashChip/SPI_MISO
- U3 pad 11: /FlashSD/SDMOSI -> /FlashChip/SPI_MOSI
- U3 pad 29: /FlashSD/SDCLK -> /FlashChip/SPICLK
- U3 pad 33: /CAN Transciever/CAN_TX_2 -> /CAN Transciever/CAN_RX_2
- U3 pad 34: /CAN Transciever/CAN_RX_2 -> /CAN Transciever/CAN_TX_2
- U3 pad 55: unconnected-(U3-PB3-Pad55) -> /MCU/SWO
- U3 pad 8: unconnected-(U3-PC0-Pad8) -> /FlashChip/ChipSelectFLash
- U3 pad 9: unconnected-(U3-PC1-Pad9) -> /FlashSD/ChipSelectSDCARD
Routing:
- net /FlashChip/SPI_MISO: track 0.00 -> 69.3 mm, vias 0 -> 5
- net /FlashChip/SPICLK: track 0.00 -> 67.6 mm, vias 0 -> 5
- net /FlashChip/SPI_MOSI: track 0.00 -> 61.1 mm, vias 0 -> 3
- net /MCU/SWO: track 0.00 -> 55.6 mm, vias 0 -> 1
- net /FlashChip/ChipSelectFLash: track 0.00 -> 50.0 mm, vias 0 -> 2
- net /MCU/Encoder-B: track 0.00 -> 48.8 mm, vias 0 -> 1
- net /MCU/Encoder-A: track 0.00 -> 48.2 mm, vias 0 -> 1
- net /FlashSD/ChipSelectSDCARD: track 0.00 -> 43.1 mm, vias 0 -> 2
- net /FlashSD/SDMISO: track 41.8 -> 0.00 mm, vias 2 -> 0
- net /FlashSD/SDMOSI: track 37.4 -> 0.00 mm, vias 2 -> 0
- net /FlashSD/SDCLK: track 22.7 -> 0.00 mm, vias 2 -> 0
- net +3.3V: track 83.9 -> 93.8 mm, vias 23 -> 26
- net Net-(J3-CLK): track 7.39 -> 0.00 mm
- net Net-(J3-DAT3/CD): track 6.83 -> 0.00 mm
- net /MCU/NRST: track 59.4 -> 66.1 mm
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