File: Schematics/CAN-Interface-Board.kicad_sch (KiCad schematic)
At the start: 4 parts, among them J6 Conn_01x05_Pin

Commit message: V2, need to add flash mem, and encoder
Other:
- added sheet FlashChip (Flash_chip.kicad_sch)
Changed lines of the file:
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@@
+	)
+	(sheet
+		(at 186.69 30.48)
+		(size 29.21 16.51)
+		(exclude_from_sim no)
+		(in_bom yes)
+		(on_board yes)
+		(dnp no)
+		(fields_autoplaced yes)
+		(stroke
+			(width 0.1524)
+			(type solid)
+		)
+		(fill
+			(color 0 0 0 0)
+		)
+		(property "Sheetname" "FlashChip"
+			(at 186.69 29.7684 0)
+			(show_name no)
+			(do_not_autoplace no)
+			(effects
+				(font
+					(size 1.27 1.27)
+				)
+				(justify left bottom)
+			)
+		)
+		(property "Sheetfile" "Flash_chip.kicad_sch"
+			(at 186.69 47.5746 0)
+			(show_name no)
+			(do_not_autoplace no)
+			(effects
+				(font
+					(size 1.27 1.27)
+				)
+				(justify left top)
+			)
+		)
+		(instances
+			(project "CAN-Interface-Board"
+				(path "/8a3e7f99-4046-40e8-bd7c-d9d1c8c7162e"
+					(page "2")
+				)
+			)
+		)
 	)
 	(sheet

Commit message: need to finish st link and flash mem layout
Other:
- sheet FlashChip ports: added ChipSelectFLash, SPICLK, SPI_MISO, SPI_MOSI; removed none
