File: Schematics/CAN-Interface-Board.kicad_sch (KiCad schematic)
At the start: 4 parts, among them J6 Conn_01x05_Pin

Commit message: pcb pending review and order
Other:
- sheet FlashChip ports: added ChipSelectFLash, SPICLK, SPI_MISO, SPI_MOSI; removed none
- sheet FlashSD ports: added ChipSelectSDCARD; removed none
- sheet MCU ports: added 5Venable, CS_FLASHMEM, CS_SDCARD; removed none
