File: Schematics/FlashSD.kicad_sch (KiCad schematic)
At the start: 3 parts, among them J3 Micro_SD_Card

Commit message: V2, need to add flash mem, and encoder
Connections:
- net SDMISO: now also J3.7 (DAT0); no longer J3.3 (CMD)
- net SDMOSI: now also J3.3 (CMD); no longer J3.7 (DAT0)
Changed lines of the file:
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@@
 	(wire
 		(pts
-			(xy 105.41 91.44) (xy 149.86 91.44)
+			(xy 147.32 93.98) (xy 149.86 93.98)
 		)
 		(stroke
@@
 	(wire
 		(pts
-			(xy 147.32 93.98) (xy 149.86 93.98)
+			(xy 105.41 91.44) (xy 149.86 91.44)
 		)
 		(stroke
@@
 	(wire
 		(pts
-			(xy 105.41 101.6) (xy 149.86 101.6)
+			(xy 115.57 96.52) (xy 149.86 96.52)
 		)
 		(stroke
@@
 	(wire
 		(pts
-			(xy 115.57 96.52) (xy 149.86 96.52)
+			(xy 105.41 101.6) (xy 149.86 101.6)
 		)
 		(stroke
@@
 	(hierarchical_label "SDMOSI"
 		(shape input)
-		(at 105.41 101.6 180)
+		(at 105.41 91.44 180)
 		(effects
 			(font
@@
 	(hierarchical_label "SDMISO"
 		(shape input)
-		(at 105.41 91.44 180)
+		(at 105.41 101.6 180)
 		(effects
 			(font

Commit message: pcb pending review and order
Parts:
- removed J3: Micro_SD_Card, Connector_Card:microSD_HC_Molex_47219-2001, symbol Connector:Micro_SD_Card
- removed R8: 33r, Resistor_SMD:R_0805_2012Metric_Pad1.20x1.40mm_HandSolder, symbol Device:R
- removed R9: 10k, Resistor_SMD:R_0805_2012Metric_Pad1.20x1.40mm_HandSolder, symbol Device:R
- added J8: Micro_SD_Card, Connector_Card:microSD_HC_Molex_47219-2001, symbol Connector:Micro_SD_Card
- added R15: 10k, Resistor_SMD:R_0805_2012Metric_Pad1.20x1.40mm_HandSolder, symbol Device:R
Connections:
- net +3.3V: now also J8.4 (VDD), R15.1
- net GND: now also J8.6 (VSS), J8.9 (SHIELD)
- net SDCLK: now also J8.5 (CLK)
- net SDMISO: now also J8.7 (DAT0)
- net SDMOSI: now also J8.3 (CMD)
- new net ChipSelectSDCARD: J8.2 (DAT3/CD), R15.2
Other:
- note added: "SD Card for flight telemetry logging and possible lookup tables for control systems"
