File: Schematics/MCU.kicad_sch (KiCad schematic)
At the start: 27 parts, among them J1 Microsemi_FlashPro-JTAG-10, U3 STM32F405RGT6, Y1 8mhz

Commit message: pcb pending review and order
Parts:
- removed J1: Microsemi_FlashPro-JTAG-10, Connector_PinHeader_1.27mm:PinHeader_2x05_P1.27mm_Vertical, symbol Connector:Microsemi_FlashPro-JTAG-10
- added J1: Conn_ARM_JTAG_SWD_10, Connector_PinHeader_1.27mm:PinHeader_2x05_P1.27mm_Vertical, symbol Custom1:Conn_ARM_JTAG_SWD_10
Connections:
- net +3.3V: now also J1.1 (VTref)
- net GND: now also J1.3 (GND), J1.5 (GND), J1.9 (GNDDetect)
- net NRST: now also J1.10 (~{RESET})
- net SWCLK: now also J1.4 (SWCLK/TCK)
- net SWDIO: now also J1.2 (SWDIO/TMS)
- net SWO: now reaches U3.55 (PB3)
- net SWO: now also J1.6 (SWO/TDO)
- net CS_FLASHMEM: now reaches U3.8 (PC0)
- net CS_SDCARD: now reaches U3.9 (PC1)
- no-connect marks 32 -> 26
