File: Schematics/Power.kicad_sch (KiCad schematic)
At the start: 6 parts, among them U2 LDL1117-3.3

Commit message: pcb pending review and order
Connections:
- net +3.3V: now also U2.2 (Vout); no longer U2.3 (Vout)
- net GND: now also U2.1 (GND); no longer U2.2 (GND)
- net at C4.1, D1.1 (K), D2.1 (K): now also U2.3 (Vin); no longer U2.1 (Vin)
Changed lines of the file:
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@@
-	(wire
-		(pts
-			(xy 96.52 120.65) (xy 100.33 120.65)
-		)
-		(stroke
-			(width 0)
-			(type default)
-		)
-	)
 	(wire
 		(pts
@@
 		)
 		(stroke
+			(width 0)
+			(type default)
+		)
+	)
+	(wire
+		(pts
+			(xy 96.52 120.65) (xy 100.33 120.65)
+		)
+		(stroke
